File: ArduinoDriverSheild/ArduinoDriverSheild.kicad_pcb (KiCad board)
At the start: 2 copper layers, 68.6 x 53.3 mm, 8 parts, among them P1 Power, P2 Analog, P3 Digital, P4 Digital, P5 CONN_01X01, P6 CONN_01X01, P7 CONN_01X01, P8 CONN_01X01

Commit message: Completed on Arduino Driver Sheild.
Parts:
- added J101: Screw_Terminal_01x02, Connectors_Terminal_Blocks:TerminalBlock_Pheonix_PT-3.5mm_2pol, F.Cu at (130.4, 120.0)
- added J102: Screw_Terminal_01x09, Connectors_Terminal_Blocks:TerminalBlock_Pheonix_PT-3.5mm_9pol, F.Cu at (166.9, 116.9)
- added U101: TBD62083A, Housings_SOIC:SOIC-18W_7.5x11.6mm_Pitch1.27mm, F.Cu at (151.6, 89.9)
Routing:
- added copper zone on F.Cu, net +VDC
- added copper zone on B.Cu, net GND
