File: ArduinoDriverSheild/ArduinoDriverSheild.kicad_pcb (KiCad board)
At the start: 2 copper layers, 68.6 x 53.3 mm, 11 parts, among them J101 Screw_Terminal_01x02, J102 Screw_Terminal_01x09, P1 Power, P2 Analog, P3 Digital, P4 Digital, P5 CONN_01X01, P6 CONN_01X01, P7 CONN_01X01, P8 CONN_01X01, U101 TBD62083A

Commit message: Completed on Arduino Driver Sheild.
Routing:
- net Net-(J102-Pad2): track 0.00 -> 37.6 mm, vias 0 -> 1
- net /2: track 0.00 -> 31.2 mm, vias 0 -> 2
- net Net-(J102-Pad3): track 0.00 -> 24.7 mm, vias 0 -> 1
- net Net-(J102-Pad9): track 0.00 -> 24.4 mm, vias 0 -> 1
- net Net-(J102-Pad4): track 0.00 -> 23.0 mm, vias 0 -> 1
- net Net-(J102-Pad5): track 0.00 -> 20.2 mm, vias 0 -> 1
- net Net-(J102-Pad8): track 0.00 -> 19.2 mm, vias 0 -> 1
- net Net-(J102-Pad6): track 0.00 -> 18.2 mm, vias 0 -> 1
- net Net-(J102-Pad7): track 0.00 -> 17.4 mm, vias 0 -> 1
- net /3(**): track 0.00 -> 14.3 mm
- net /4: track 0.00 -> 13.4 mm
- net /5(**): track 0.00 -> 12.9 mm
- net /7: track 0.00 -> 12.6 mm
- net /6(**): track 0.00 -> 12.4 mm
- net /8: track 0.00 -> 10.7 mm
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Changed lines of the file:
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@@
   (general
     (links 24)
-    (no_connects 23)
+    (no_connects 2)
     (area 110.922999 72.949999 179.653001 126.440001)
     (thickness 1.6)
     (drawings 27)
-    (tracks 0)
+    (tracks 67)
     (zones 0)
     (modules 11)
@@
   )
   (setup
-    (last_trace_width 0.25)
+    (last_trace_width 0.5)
+    (user_trace_width 0.5)
     (trace_clearance 0.2)
     (zone_clearance 0.508)
@@
     (via_min_size 0.4)
     (via_min_drill 0.3)
+    (user_via 1.2 0.8)
     (uvia_size 0.3)
     (uvia_drill 0.1)
@@
   (gr_line (start 120.523 82.55) (end 120.523 93.98) (angle 90) (layer Dwgs.User) (width 0.15))
   (gr_line (start 104.648 82.55) (end 120.523 82.55) (angle 90) (layer Dwgs.User) (width 0.15))
+  (segment (start 146.558 85.215) (end 146.558 83.185) (width 0.5) (layer F.Cu) (net 4))
+  (via (at 146.558 83.185) (size 1.2) (drill 0.8) (layers F.Cu B.Cu) (net 4))
+  (segment (start 149.098 85.215) (end 149.098 76.581) (width 0.5) (layer F.Cu) (net 13))
+  (segment (start 149.098 76.581) (end 150.114 75.565) (width 0.5) (layer F.Cu) (net 13))
+  (segment (start 150.368 85.215) (end 150.368 77.851) (width 0.5) (layer F.Cu) (net 14))
+  (segment (start 150.368 77.851) (end 151.138 77.081) (width 0.5) (layer F.Cu) (net 14))
+  (segment (start 151.138 77.081) (end 151.2904 77.081) (width 0.5) (layer F.Cu) (net 14))
+  (segment (start 151.2904 77.081) (end 152.654 75.7174) (width 0.5) (layer F.Cu) (net 14))
+  (segment (start 152.654 75.7174) (end 152.654 75.565) (width 0.5) (layer F.Cu) (net 14))
+  (segment (start 151.638 85.215) (end 151.638 79.2814) (width 0.5) (layer F.Cu) (net 15))
+  (segment (start 151.638 79.2814) (end 155.3544 75.565) (width 0.5) (layer F.Cu) (net 15))
+  (segment (start 155.3544 75.565) (end 156.718 75.565) (width 0.5) (layer F.Cu) (net 15))
+  (segment (start 152.908 85.215) (end 152.908 81.915) (width 0.5) (layer F.Cu) (net 16))
+  (segment (start 152.908 81.915) (end 157.742 77.081) (width 0.5) (layer F.Cu) (net 16))
+  (segment (start 159.258 75.7174) (end 159.258 75.565) (width 0.5) (layer F.Cu) (net 16))
+  (segment (start 157.742 77.081) (end 157.8944 77.081) (width 0.5) (layer F.Cu) (net 16))
+  (segment (start 157.8944 77.081) (end 159.258 75.7174) (width 0.5) (layer F.Cu) (net 16))
+  (segment (start 154.178 85.215) (end 154.178 83.185) (width 0.5) (layer F.Cu) (net 17))
+  (segment (start 154.178 83.185) (end 160.282 77.081) (width 0.5) (layer F.Cu) (net 17))
+  (segment (start 160.282 77.081) (end 160.4344 77.081) (width 0.5) (layer F.Cu) (net 17))
+  (segment (start 160.4344 77.081) (end 161.798 75.7174) (width 0.5) (layer F.Cu) (net 17))
+  (segment (start 161.798 75.7174) (end 161.798 75.565) (width 0.5) (layer F.Cu) (net 17))
+  (segment (start 155.448 85.215) (end 155.448 84.515) (width 0.5) (layer F.Cu) (net 18))
+  (segment (start 162.9744 77.081) (end 164.338 75.7174) (width 0.5) (layer F.Cu) (net 18))
+  (segment (start 155.448 84.515) (end 162.882 77.081) (width 0.5) (layer F.Cu) (net 18))
+  (segment (start 162.882 77.081) (end 162.9744 77.081) (width 0.5) (layer F.Cu) (net 18))
+  (segment (start 164.338 75.7174) (end 164.338 75.565) (width 0.5) (layer F.Cu) (net 18))
+  (segment (start 156.718 85.215) (end 157.518 85.215) (width 0.5) (layer F.Cu) (net 19))
+  (segment (start 157.518 85.215) (end 166.878 75.855) (width 0.5) (layer F.Cu) (net 19))
+  (segment (start 166.878 75.855) (end 166.878 75.565) (width 0.5) (layer F.Cu) (net 19))
+  (segment (start 169.418 78.105) (end 169.418 75.565) (width 0.5) (layer F.Cu) (net 20))
+  (segment (start 147.828 78.105) (end 169.418 78.105) (width 0.5) (layer B.Cu) (net 20))
+  (via (at 169.418 78.105) (size 1.2) (drill 0.8) (layers F.Cu B.Cu) (net 20))
+  (segment (start 147.828 85.215) (end 147.828 78.105) (width 0.5) (layer F.Cu) (net 20))
+  (via (at 147.828 78.105) (size 1.2) (drill 0.8) (layers F.Cu B.Cu) (net 20))
+  (segment (start 147.828 113.03) (end 147.828 94.615) (width 0.5) (layer F.Cu) (net 34))
+  (segment (start 148.183 113.385) (end 147.828 113.03) (width 0.5) (layer B.Cu) (net 34))
+  (via (at 147.828 113.03) (size 1.2) (drill 0.8) (layers F.Cu B.Cu) (net 34))
+  (segment (start 166.878 113.385) (end 148.183 113.385) (width 0.5) (layer B.Cu) (net 34))
+  (segment (start 156.718 108.585) (end 156.718 94.615) (width 0.5) (layer F.Cu) (net 35))
+  (segment (start 166.878 109.885) (end 158.018 109.885) (width 0.5) (layer B.Cu) (net 35))
+  (segment (start 158.018 109.885) (end 156.718 108.585) (width 0.5) (layer B.Cu) (net 35))
+  (via (at 156.718 108.585) (size 1.2) (drill 0.8) (layers F.Cu B.Cu) (net 35))
+  (segment (start 155.448 106.045) (end 155.448 94.615) (width 0.5) (layer F.Cu) (net 36))
+  (segment (start 166.878 106.385) (end 155.788 106.385) (width 0.5) (layer B.Cu) (net 36))
+  (segment (start 155.788 106.385) (end 155.448 106.045) (width 0.5) (layer B.Cu) (net 36))
+  (via (at 155.448 106.045) (size 1.2) (drill 0.8) (layers F.Cu B.Cu) (net 36))
+  (segment (start 154.178 101.6) (end 154.178 94.615) (width 0.5) (layer F.Cu) (net 37))
+  (segment (start 166.878 102.885) (end 155.463 102.885) (width 0.5) (layer B.Cu) (net 37))
+  (segment (start 155.463 102.885) (end 154.178 101.6) (width 0.5) (layer B.Cu) (net 37))
+  (via (at 154.178 101.6) (size 1.2) (drill 0.8) (layers F.Cu B.Cu) (net 37))
+  (segment (start 152.908 98.425) (end 152.908 94.615) (width 0.5) (layer F.Cu) (net 38))
+  (segment (start 166.878 99.385) (end 153.868 99.385) (width 0.5) (layer B.Cu) (net 38))
+  (segment (start 153.868 99.385) (end 152.908 98.425) (width 0.5) (layer B.Cu) (net 38))
+  (via (at 152.908 98.425) (size 1.2) (drill 0.8) (layers F.Cu B.Cu) (net 38))
+  (segment (start 151.638 96.52) (end 151.638 94.615) (width 0.5) (layer F.Cu) (net 39))
+  (segment (start 166.878 95.885) (end 152.273 95.885) (width 0.5) (layer B.Cu) (net 39))
+  (segment (start 152.273 95.885) (end 151.638 96.52) (width 0.5) (layer B.Cu) (net 39))
+  (via (at 151.638 96.52) (size 1.2) (drill 0.8) (layers F.Cu B.Cu) (net 39))
+  (segment (start 150.368 92.075) (end 150.368 94.615) (width 0.5) (layer F.Cu) (net 40))
+  (segment (start 166.878 92.385) (end 150.678 92.385) (width 0.5) (layer B.Cu) (net 40))
+  (segment (start 150.678 92.385) (end 150.368 92.075) (width 0.5) (layer B.Cu) (net 40))
+  (via (at 150.368 92.075) (size 1.2) (drill 0.8) (layers F.Cu B.Cu) (net 40))
+  (segment (start 149.098 88.265) (end 149.098 94.615) (width 0.5) (layer F.Cu) (net 41))
+  (segment (start 166.878 88.885) (end 149.718 88.885) (width 0.5) (layer B.Cu) (net 41))
+  (segment (start 149.718 88.885) (end 149.098 88.265) (width 0.5) (layer B.Cu) (net 41))
+  (via (at 149.098 88.265) (size 1.2) (drill 0.8) (layers F.Cu B.Cu) (net 41))
   (zone (net 33) (net_name +VDC) (layer F.Cu) (hatch edge 0.508)
     (connect_pads yes (clearance 0.508))
     (min_thickness 0.254)
-    (fill (arc_segments 16) (thermal_gap 0.508) (thermal_bridge_width 0.508))
+    (fill yes (arc_segments 16) (thermal_gap 0.508) (thermal_bridge_width 0.508))
     (polygon
       (pts
@@
     (connect_pads yes (clearance 0.508))
     (min_thickness 0.254)
-    (fill (arc_segments 16) (thermal_gap 0.508) (thermal_bridge_width 0.508))
+    (fill yes (arc_segments 16) (thermal_gap 0.508) (thermal_bridge_width 0.508))
     (polygon
       (pts
