File: ArduinoDriverSheild/ArduinoDriverSheild.sch (KiCad schematic (older format))
At the start: 18 parts, among them P1 Power, P2 Analog, P3 Digital, P4 Digital, P5 CONN_01X01, P6 CONN_01X01, P7 CONN_01X01, P8 CONN_01X01

Commit message: Completed on Arduino Driver Sheild.
Parts:
- J101: renamed from J?; footprint (none) -> Connectors_Terminal_Blocks:TerminalBlock_Pheonix_PT-3.5mm_2pol
- J102: renamed from J?; footprint (none) -> Connectors_Terminal_Blocks:TerminalBlock_Pheonix_PT-3.5mm_9pol
- U101: renamed from U?; footprint (none) -> Housings_SOIC:SOIC-18W_7.5x11.6mm_Pitch1.27mm
- gave numbers to parts that had none: 1
Connections:
- net 2: now also U101.8 (In); no longer U101.1 (In)
- net 3(**): now also U101.1 (In); no longer U101.2 (In)
- net 4: now also U101.2 (In); no longer U101.3 (In)
- net 5(**): now also U101.3 (In); no longer U101.4 (In)
- net 6(**): now also U101.4 (In); no longer U101.5 (In)
- net 7: now also U101.5 (In); no longer U101.6 (In)
- net 8: now also U101.6 (In); no longer U101.7 (In)
- net 9(**): now also U101.7 (In); no longer U101.8 (In)
- net at J102.2 (Pin_2): now also U101.11 (Out); no longer U101.18 (Out)
- net at J102.3 (Pin_3): now also U101.18 (Out); no longer U101.17 (Out)
- net at J102.4 (Pin_4): now also U101.17 (Out); no longer U101.16 (Out)
- net at J102.5 (Pin_5): now also U101.16 (Out); no longer U101.15 (Out)
- net at J102.6 (Pin_6): now also U101.15 (Out); no longer U101.14 (Out)
- net at J102.7 (Pin_7): now also U101.14 (Out); no longer U101.13 (Out)
- net at J102.8 (Pin_8): now also U101.13 (Out); no longer U101.12 (Out)
- net at J102.9 (Pin_9): now also U101.12 (Out); no longer U101.11 (Out)
Changed lines of the file:
@@
 Reset
 $Comp
-L +3.3V #PWR01
+L +3.3V #PWR107
 U 1 1 56D70538
 P 9150 1450
-F 0 "#PWR01" H 9150 1300 50  0001 C CNN
+F 0 "#PWR107" H 9150 1300 50  0001 C CNN
 F 1 "+3.3V" H 9150 1590 50  0000 C CNN
 F 2 "" H 9150 1450 50  0000 C CNN
@@
 $EndComp
 $Comp
-L +5V #PWR02
+L +5V #PWR106
 U 1 1 56D707BB
 P 9050 1350
-F 0 "#PWR02" H 9050 1200 50  0001 C CNN
+F 0 "#PWR106" H 9050 1200 50  0001 C CNN
 F 1 "+5V" H 9050 1490 50  0000 C CNN
 F 2 "" H 9050 1350 50  0000 C CNN
@@
 $EndComp
 $Comp
-L GND #PWR03
+L GND #PWR108
 U 1 1 56D70CC2
 P 9300 3150
-F 0 "#PWR03" H 9300 2900 50  0001 C CNN
+F 0 "#PWR108" H 9300 2900 50  0001 C CNN
 F 1 "GND" H 9300 3000 50  0000 C CNN
 F 2 "" H 9300 3150 50  0000 C CNN
@@
 $EndComp
 $Comp
-L GND #PWR04
+L GND #PWR109
 U 1 1 56D70CFF
 P 10300 3150
-F 0 "#PWR04" H 10300 2900 50  0001 C CNN
+F 0 "#PWR109" H 10300 2900 50  0001 C CNN
 F 1 "GND" H 10300 3000 50  0000 C CNN
 F 2 "" H 10300 3150 50  0000 C CNN
@@
 1
 $Comp
-L TBD62083A U?
-U 1 1 63DFA5B1
+L TBD62083A U101
+U 8 1 63DFA5B1
 P 3475 3075
-F 0 "U?" H 3575 2925 60  0000 C CNN
+F 0 "U101" H 3575 2925 60  0000 C CNN
 F 1 "TBD62083A" H 3725 3175 60  0000 C CNN
-F 2 "" H 3475 3075 60  0000 C CNN
+F 2 "Housings_SOIC:SOIC-18W_7.5x11.6mm_Pitch1.27mm" H 3475 3075 60  0001 C CNN
 F 3 "" H 3475 3075 60  0000 C CNN
-	1    3475 3075
-	1    0    0    -1
-$EndComp
-$Comp
-L +VDC #PWR?
+	8    3475 3075
+	1    0    0    -1
+$EndComp
+$Comp
+L +VDC #PWR101
 U 1 1 63DFA627
 P 3475 2875
-F 0 "#PWR?" H 3475 2775 50  0001 C CNN
+F 0 "#PWR101" H 3475 2775 50  0001 C CNN
 F 1 "+VDC" H 3475 3125 50  0000 C CNN
 F 2 "" H 3475 2875 50  0001 C CNN
@@
 $EndComp
 $Comp
-L GND #PWR?
+L GND #PWR102
 U 1 1 63DFA6BA
 P 3475 3275
-F 0 "#PWR?" H 3475 3025 50  0001 C CNN
+F 0 "#PWR102" H 3475 3025 50  0001 C CNN
 F 1 "GND" H 3475 3125 50  0000 C CNN
 F 2 "" H 3475 3275 50  0001 C CNN
@@
 $EndComp
 $Comp
-L TBD62083A U?
-U 2 1 63DFA717
+L TBD62083A U101
+U 1 1 63DFA717
 P 3450 3725
-F 0 "U?" H 3550 3575 60  0000 C CNN
+F 0 "U101" H 3550 3575 60  0000 C CNN
 F 1 "TBD62083A" H 3700 3825 60  0000 C CNN
 F 2 "" H 3450 3725 60  0000 C CNN
 F 3 "" H 3450 3725 60  0000 C CNN
-	2    3450 3725
-	1    0    0    -1
-$EndComp
-$Comp
-L TBD62083A U?
-U 3 1 63DFA7BE
+	1    3450 3725
+	1    0    0    -1
+$EndComp
+$Comp
+L TBD62083A U101
+U 2 1 63DFA7BE
 P 3450 4200
-F 0 "U?" H 3550 4050 60  0000 C CNN
+F 0 "U101" H 3550 4050 60  0000 C CNN
 F 1 "TBD62083A" H 3700 4300 60  0000 C CNN
 F 2 "" H 3450 4200 60  0000 C CNN
 F 3 "" H 3450 4200 60  0000 C CNN
-	3    3450 4200
-	1    0    0    -1
-$EndComp
-$Comp
-L TBD62083A U?
-U 4 1 63DFA81C
+	2    3450 4200
+	1    0    0    -1
+$EndComp
+$Comp
+L TBD62083A U101
+U 3 1 63DFA81C
 P 3450 4700
-F 0 "U?" H 3550 4550 60  0000 C CNN
+F 0 "U101" H 3550 4550 60  0000 C CNN
 F 1 "TBD62083A" H 3700 4800 60  0000 C CNN
 F 2 "" H 3450 4700 60  0000 C CNN
 F 3 "" H 3450 4700 60  0000 C CNN
-	4    3450 4700
-	1    0    0    -1
-$EndComp
-$Comp
-L TBD62083A U?
-U 5 1 63DFA89D
+	3    3450 4700
+	1    0    0    -1
+$EndComp
+$Comp
+L TBD62083A U101
+U 4 1 63DFA89D
 P 3450 5200
-F 0 "U?" H 3550 5050 60  0000 C CNN
+F 0 "U101" H 3550 5050 60  0000 C CNN
 F 1 "TBD62083A" H 3700 5300 60  0000 C CNN
 F 2 "" H 3450 5200 60  0000 C CNN
 F 3 "" H 3450 5200 60  0000 C CNN
-	5    3450 5200
-	1    0    0    -1
-$EndComp
-$Comp
-L TBD62083A U?
-U 6 1 63DFA95B
+	4    3450 5200
+	1    0    0    -1
+$EndComp
+$Comp
+L TBD62083A U101
+U 5 1 63DFA95B
 P 3450 5650
-F 0 "U?" H 3550 5500 60  0000 C CNN
+F 0 "U101" H 3550 5500 60  0000 C CNN
 F 1 "TBD62083A" H 3700 5750 60  0000 C CNN
 F 2 "" H 3450 5650 60  0000 C CNN
 F 3 "" H 3450 5650 60  0000 C CNN
-	6    3450 5650
-	1    0    0    -1
-$EndComp
-$Comp
-L TBD62083A U?
-U 7 1 63DFA9C8
+	5    3450 5650
+	1    0    0    -1
+$EndComp
+$Comp
+L TBD62083A U101
+U 6 1 63DFA9C8
 P 3450 6150
-F 0 "U?" H 3550 6000 60  0000 C CNN
+F 0 "U101" H 3550 6000 60  0000 C CNN
 F 1 "TBD62083A" H 3700 6250 60  0000 C CNN
 F 2 "" H 3450 6150 60  0000 C CNN
 F 3 "" H 3450 6150 60  0000 C CNN
-	7    3450 6150
-	1    0    0    -1
-$EndComp
-$Comp
-L TBD62083A U?
-U 8 1 63DFAAAB
+	6    3450 6150
+	1    0    0    -1
+$EndComp
+$Comp
+L TBD62083A U101
+U 7 1 63DFAAAB
 P 3450 6725
-F 0 "U?" H 3550 6575 60  0000 C CNN
+F 0 "U101" H 3550 6575 60  0000 C CNN
 F 1 "TBD62083A" H 3700 6825 60  0000 C CNN
 F 2 "" H 3450 6725 60  0000 C CNN
 F 3 "" H 3450 6725 60  0000 C CNN
-	8    3450 6725
+	7    3450 6725
 	1    0    0    -1
 $EndComp
@@
 9(**)
 $Comp
-L Screw_Terminal_01x09 J?
+L Screw_Terminal_01x09 J102
 U 1 1 63DFC18D
 P 5200 3750
-F 0 "J?" H 5200 4250 50  0000 C CNN
+F 0 "J102" H 5200 4250 50  0000 C CNN
 F 1 "Screw_Terminal_01x09" H 5200 3250 50  0000 C CNN
-F 2 "" H 5200 3750 50  0001 C CNN
+F 2 "Connectors_Terminal_Blocks:TerminalBlock_Pheonix_PT-3.5mm_9pol" H 5200 3750 50  0001 C CNN
 F 3 "" H 5200 3750 50  0001 C CNN
 	1    5200 3750
@@
 $EndComp
 $Comp
-L Screw_Terminal_01x02 J?
+L Screw_Terminal_01x02 J101
 U 1 1 63DFC3C2
 P 5200 2650
-F 0 "J?" H 5200 2750 50  0000 C CNN
+F 0 "J101" H 5200 2750 50  0000 C CNN
 F 1 "Screw_Terminal_01x02" H 5200 2450 50  0000 C CNN
-F 2 "" H 5200 2650 50  0001 C CNN
+F 2 "Connectors_Terminal_Blocks:TerminalBlock_Pheonix_PT-3.5mm_2pol" H 5200 2650 50  0001 C CNN
 F 3 "" H 5200 2650 50  0001 C CNN
 	1    5200 2650
@@
 $EndComp
 $Comp
-L +VDC #PWR?
+L +VDC #PWR103
 U 1 1 63DFC489
 P 5000 2650
-F 0 "#PWR?" H 5000 2550 50  0001 C CNN
+F 0 "#PWR103" H 5000 2550 50  0001 C CNN
 F 1 "+VDC" H 5000 2900 50  0000 C CNN
 F 2 "" H 5000 2650 50  0001 C CNN
@@
 $EndComp
 $Comp
-L GND #PWR?
+L GND #PWR104
 U 1 1 63DFC4CA
 P 5000 2750
-F 0 "#PWR?" H 5000 2500 50  0001 C CNN
+F 0 "#PWR104" H 5000 2500 50  0001 C CNN
 F 1 "GND" H 5000 2600 50  0000 C CNN
 F 2 "" H 5000 2750 50  0001 C CNN
@@
 $EndComp
 $Comp
-L +VDC #PWR?
+L +VDC #PWR105
 U 1 1 63DFC51D
 P 5000 3350
-F 0 "#PWR?" H 5000 3250 50  0001 C CNN
+F 0 "#PWR105" H 5000 3250 50  0001 C CNN
 F 1 "+VDC" H 5000 3600 50  0000 C CNN
 F 2 "" H 5000 3350 50  0001 C CNN
