File: 6footfl/6footfl.kicad_pcb (KiCad board)
At the start: 2 copper layers, 21 x 1.8 mm, 6 parts, among them J101 -, J102 +

Commit message: Upgrade Kicad version.
Other:
- net class Default removed
