File: 8BallSign/8BallLEDPCB.kicad_pcb (KiCad board)
At the start: 2 copper layers, 31.8 x 76.2 mm, 41 parts, among them J101 Solder pads

Commit message: Upgrade Kicad version.
Other:
- net class Default removed
