File: BarOverhead/BarOverhead.kicad_pcb (KiCad board)
At the start: 2 copper layers, 88.9 x 12.7 mm, 6 parts, among them J101 -, J102 +

Commit message: Upgrade Kicad version.
Other:
- net class Default removed
