File: MovieTheaterMarque/MovieTheaterMarque.kicad_pcb (KiCad board)
At the start: 2 copper layers, 64 x 14 mm, 50 parts, among them J101 Input, J102 Output, U101 ws2812b-2020, U102 ws2812b-2020, U103 ws2812b-2020, U104 ws2812b-2020, U105 ws2812b-2020, U106 ws2812b-2020, U107 ws2812b-2020, U108 ws2812b-2020, U109 ws2812b-2020, U110 ws2812b-2020, U111 ws2812b-2020, U112 ws2812b-2020, U113 ws2812b-2020, U114 ws2812b-2020, U115 ws2812b-2020, U116 ws2812b-2020, U117 ws2812b-2020, U118 ws2812b-2020, U119 ws2812b-2020, U120 ws2812b-2020, U121 ws2812b-2020, U122 ws2812b-2020, U123 ws2812b-2020, U124 ws2812b-2020, U126 ws2812b-2020, U127 ws2812b-2020, U128 ws2812b-2020, U130 ws2812b-2020, U131 ws2812b-2020, U132 ws2812b-2020, U134 ws2812b-2020, U135 ws2812b-2020, U136 ws2812b-2020, U138 ws2812b-2020, U139 ws2812b-2020, U140 ws2812b-2020, U142 ws2812b-2020, U143 ws2812b-2020, U144 ws2812b-2020, U146 ws2812b-2020, U147 ws2812b-2020, U148 ws2812b-2020, U150 ws2812b-2020, U151 ws2812b-2020, U152 ws2812b-2020, U154 ws2812b-2020, U155 ws2812b-2020, U156 ws2812b-2020

Commit message: Upgrade Kicad version.
Other:
- net class Default removed
